Commit message: stick URDF

File: rl_crazyflie/assets/stick.urdf (robot description, URDF)
Before this commit: robot stick, 1 links, 0 joints
Links:
- added link top, mass 0.0027; collision sphere radius=0.02; visual sphere radius=0.02
Joints:
- added joint joint1: type fixed, parent base_link, child top, origin xyz=0 0 0 rpy=0 0 0

File: rl_crazyflie/assets/stick.xacro (robot description, xacro)
@@ -3,18 +3,19 @@
     <xacro:property name="cylinderLength" value="0.3" />
     <xacro:property name="cylinderRadius" value="0.005" />
+    <xacro:property name="cylinderMass" value="0.0027" />
     <link name="base_link">
         <visual>
             <!-- with respect to the center of the cylinder -->
-            <origin rpy="0 0 0" xyz="0 0 0"/>
+            <origin rpy="0 0 0" xyz="0 0 ${cylinderLength/2}"/>
             <geometry>
                 <cylinder length="${cylinderLength}" radius="${cylinderRadius}" />
             </geometry>
-            <material name="red">
-                <color rgba="0.8 0 0 1" />
+            <material name="gray">
+                <color rgba="0.5 0.5 0.5 1" />
             </material>
         </visual>
         <!-- similar to visual, can be different for safer zones/computation -->
         <collision>
-            <origin rpy="0 0 0" xyz="0 0 0"/>
+            <origin rpy="0 0 0" xyz="0 0 ${cylinderLength/2}"/>
             <geometry>
                 <cylinder length="${cylinderLength}" radius="${cylinderRadius}" />
@@ -22,10 +23,43 @@
         </collision>
         <inertial>
-            <origin rpy="0 0 0" xyz="0 0 0"/>
+            <origin rpy="0 0 0" xyz="0 0 ${cylinderLength/2}"/>
             <!-- in kgs -->
-            <mass value="0.0027"/>
+            <mass value="${cylinderMass}"/>
             <!-- calc from script -->
             <inertia ixx="2.0e-5" ixy="0.0" ixz="0.0" iyy="2.0e-5" iyz="0.0" izz="3.3e-8"/>
         </inertial>
     </link>
+    <xacro:property name="sphereRadius" value="0.02" />
+    <xacro:property name="sphereMass" value="0.0027" />
+    <link name="top">
+        <visual>
+            <!-- shift origin to the top -->
+            <origin rpy="0 0 0" xyz="0 0 ${cylinderLength}" />
+            <geometry>
+                <sphere radius="${sphereRadius}" />
+            </geometry>
+            <material name="red">
+                <color rgba="1 0 0 1" />
+            </material>
+        </visual>
+        <collision>
+            <origin rpy="0 0 0" xyz="0 0 ${cylinderLength}" />
+            <geometry>
+                <sphere radius="${sphereRadius}" />
+            </geometry>
+        </collision>
+        <inertial>
+            <origin rpy="0 0 0" xyz="0 0 ${cylinderLength}"/>
+            <!-- in kgs -->
+            <mass value="${sphereMass}"/>
+            <!-- calc from script -->
+            <inertia ixx="7.2e-7" ixy="0.0" ixz="0.0" iyy="7.2e-7" iyz="0.0" izz="7.2e-7"/>
+        </inertial>
+    </link>
+    <joint name="joint1" type="fixed">
+        <parent link="base_link"/>
+        <child link="top"/>
+        <!-- with respect the parent reference -->
+        <origin rpy="0 0 0" xyz="0 0 0" />
+    </joint>
 </robot>

Commit message: URDF: fixed stick origin

File: rl_crazyflie/assets/stick.urdf (robot description, URDF)
Before this commit: robot stick, 2 links, 1 joints
Links:
- removed link base_link
- added link base, mass 0.0027; collision cylinder length=0.3 radius=0.005; visual cylinder length=0.3 radius=0.005
Joints:
- joint joint1: child top -> base; parent base_link -> top

File: rl_crazyflie/assets/stick.xacro (robot description, xacro)
@@ -4,5 +4,5 @@
     <xacro:property name="cylinderRadius" value="0.005" />
     <xacro:property name="cylinderMass" value="0.0027" />
-    <link name="base_link">
+    <link name="base">
         <visual>
             <!-- with respect to the center of the cylinder -->
@@ -58,6 +58,6 @@
     </link>
     <joint name="joint1" type="fixed">
-        <parent link="base_link"/>
-        <child link="top"/>
+        <parent link="top"/>
+        <child link="base"/>
         <!-- with respect the parent reference -->
         <origin rpy="0 0 0" xyz="0 0 0" />

Commit message: attempt 1

File: rl_crazyflie/assets/stick.urdf (robot description, URDF)
Before this commit: robot stick, 2 links, 1 joints
Links:
- link base: mass 0.0027 -> 0.001; geometry collision cylinder length=1.0 radius=0.01; visual cylinder length=1.0 radius=0.01
- link top: mass 0.0027 -> 0.003

File: rl_crazyflie/assets/stick.xacro (robot description, xacro)
@@ -1,7 +1,10 @@
 <?xml version="1.0"?>
 <robot name="stick" xmlns:xacro="http://www.ros.org/wiki/xacro">
-    <xacro:property name="cylinderLength" value="0.3" />
-    <xacro:property name="cylinderRadius" value="0.005" />
-    <xacro:property name="cylinderMass" value="0.0027" />
+    <xacro:property name="cylinderLength" value="1.0" />
+    <xacro:property name="cylinderRadius" value="0.01" />
+    <xacro:property name="cylinderMass" value="0.001" />
+    <xacro:property name="cylinderIxx" value="${1/12 * cylinderMass * (3 * cylinderRadius**2 + cylinderLength**2)}" />
+    <xacro:property name="cylinderIyy" value="${1/12 * cylinderMass * (3 * cylinderRadius**2 + cylinderLength**2)}" />
+    <xacro:property name="cylinderIzz" value="${1/2 * cylinderMass * cylinderRadius**2}" />
     <link name="base">
         <visual>
@@ -27,9 +30,12 @@
             <mass value="${cylinderMass}"/>
             <!-- calc from script -->
-            <inertia ixx="2.0e-5" ixy="0.0" ixz="0.0" iyy="2.0e-5" iyz="0.0" izz="3.3e-8"/>
+            <inertia ixx="${cylinderIxx}" ixy="0.0" ixz="0.0" iyy="${cylinderIyy}" iyz="0.0" izz="${cylinderIzz}"/>
         </inertial>
     </link>
     <xacro:property name="sphereRadius" value="0.02" />
-    <xacro:property name="sphereMass" value="0.0027" />
+    <xacro:property name="sphereMass" value="0.003" />
+    <xacro:property name="sphereIxx" value="${2/3 * sphereMass * sphereRadius**2}" />
+    <xacro:property name="sphereIyy" value="${2/3 * sphereMass * sphereRadius**2}" />
+    <xacro:property name="sphereIzz" value="${2/3 * sphereMass * sphereRadius**2}" />
     <link name="top">
         <visual>
@@ -54,5 +60,5 @@
             <mass value="${sphereMass}"/>
             <!-- calc from script -->
-            <inertia ixx="7.2e-7" ixy="0.0" ixz="0.0" iyy="7.2e-7" iyz="0.0" izz="7.2e-7"/>
+            <inertia ixx="${sphereIxx}" ixy="0.0" ixz="0.0" iyy="${sphereIyy}" iyz="0.0" izz="${sphereIzz}"/>
         </inertial>
     </link>

Commit message: works 2

File: rl_crazyflie/assets/stick.urdf (robot description, URDF)
Before this commit: robot stick, 2 links, 1 joints
Links:
- link base: mass 0.001 -> 0.002; geometry collision cylinder length=1.0 radius=0.005; visual cylinder length=1.0 radius=0.005
- link top: mass 0.003 -> 0.006; geometry collision sphere radius=0.03; visual sphere radius=0.03

File: rl_crazyflie/assets/stick.xacro (robot description, xacro)
@@ -2,6 +2,6 @@
 <robot name="stick" xmlns:xacro="http://www.ros.org/wiki/xacro">
     <xacro:property name="cylinderLength" value="1.0" />
-    <xacro:property name="cylinderRadius" value="0.01" />
-    <xacro:property name="cylinderMass" value="0.001" />
+    <xacro:property name="cylinderRadius" value="0.005" />
+    <xacro:property name="cylinderMass" value="0.002" />
     <xacro:property name="cylinderIxx" value="${1/12 * cylinderMass * (3 * cylinderRadius**2 + cylinderLength**2)}" />
     <xacro:property name="cylinderIyy" value="${1/12 * cylinderMass * (3 * cylinderRadius**2 + cylinderLength**2)}" />
@@ -33,6 +33,6 @@
         </inertial>
     </link>
-    <xacro:property name="sphereRadius" value="0.02" />
-    <xacro:property name="sphereMass" value="0.003" />
+    <xacro:property name="sphereRadius" value="0.03" />
+    <xacro:property name="sphereMass" value="0.006" />
     <xacro:property name="sphereIxx" value="${2/3 * sphereMass * sphereRadius**2}" />
     <xacro:property name="sphereIyy" value="${2/3 * sphereMass * sphereRadius**2}" />
